Commit message: Add elevator

File: models/rotors_description/urdf/fixedwing_base.xacro (robot description, xacro)
@@ -192,5 +192,5 @@
   <!-- Rotor joint and link -->
   <xacro:macro name="control_surface"
-    params="robot_namespace link_name parent color mesh_file mesh_scale *origin *axis *mesh_origin">
+    params="robot_namespace link_name parent color mesh_file mesh_scale area *origin *axis *mesh_origin">
     <joint name="${link_name}_joint" type="revolute">
       <xacro:insert_block name="origin" />
@@ -228,13 +228,13 @@
             <cma_stall>0</cma_stall>
             <cp>-0.05 0.3 0.05</cp>
-            <area>0.12</area>
+            <area>${area}</area>
             <air_density>1.2041</air_density>
             <forward>1 0 0</forward>
             <upward>0 0 1</upward>
-            <link_name>base_link</link_name>
+            <link_name>${parent}</link_name>
             <control_joint_name>
                ${link_name}_joint
             </control_joint_name>
-            <control_joint_rad_to_cl>-0.5</control_joint_rad_to_cl>
+            <control_joint_rad_to_cl>-1.0</control_joint_rad_to_cl>
          </plugin>
     </gazebo>

File: models/rotors_description/urdf/standard_vtol.xacro (robot description, xacro)
@@ -150,6 +150,6 @@
     time_constant_up="${time_constant_up}"
     time_constant_down="${time_constant_down}"
-    max_rot_velocity="${max_rot_velocity}"
-    motor_number="5"
+    max_rot_velocity="3500"
+    motor_number="4"
     rotor_drag_coefficient="${rotor_drag_coefficient}"
     rolling_moment_coefficient="${rolling_moment_coefficient}"
@@ -170,4 +170,5 @@
     mesh_file="model://standard_vtol/meshes/x8_elevon_left.dae"
     mesh_scale="0.001 0.001 0.001"
+    area="0.5"
     color="Blue">
     <origin xyz="0.0 0.65 0.0" rpy="0 0 0" />
@@ -185,4 +186,5 @@
     mesh_file="model://standard_vtol/meshes/x8_elevon_right.dae"
     mesh_scale="0.001 0.001 0.001"
+    area="0.5"
     color="Blue">
     <origin xyz="0.0 -0.65 0.0" rpy="0 0 0" />
@@ -190,3 +192,15 @@
     <xacro:insert_block name="right_elevon_mesh_origin" />
   </xacro:control_surface>
+  <xacro:control_surface
+    robot_namespace="${namespace}"
+    link_name="elevator"
+    parent="base_link"
+    mesh_file="model://standard_vtol/meshes/x8_elevon_right.dae"
+    mesh_scale="0.001 0.001 0.001"
+    area="0.5"
+    color="Blue">
+    <origin xyz="-1.0 0.0 0.0" rpy="0 0 0" />
+    <axis xyz="0 1 0" />
+    <xacro:insert_block name="right_elevon_mesh_origin" />
+  </xacro:control_surface>
 </robot>

Commit message: Decrease rudder lift coefficients

File: models/rotors_description/urdf/fixedwing_base.xacro (robot description, xacro)
@@ -119,5 +119,5 @@
   <!-- Rotor joint and link -->
   <xacro:macro name="control_surface"
-    params="robot_namespace link_name parent color mesh_file mesh_scale area control_joint_rad_to_cl a0 cpx cpy cpz upx upy upz *origin *joint_origin *axis *mesh_origin">
+    params="robot_namespace link_name parent color mesh_file mesh_scale area joint_limit control_joint_rad_to_cl a0 cpx cpy cpz upx upy upz *origin *joint_origin *axis *mesh_origin">
     <joint name="${link_name}_joint" type="revolute">
       <xacro:insert_block name="joint_origin" />
@@ -126,5 +126,5 @@
       <!-- <axis xyz="0 0 1" /> -->
       <xacro:insert_block name="axis" />
-      <limit effort="1000" velocity="1000.0" lower="-0.53" upper="0.53" />
+      <limit effort="1000" velocity="1000.0" lower="-${joint_limit}" upper="${joint_limit}" />
       <!-- <dynamics damping="1.0"/> -->
     </joint>

File: models/rotors_description/urdf/plane.xacro (robot description, xacro)
@@ -108,5 +108,6 @@
     upx="0"
     upy="0"
-    upz="1">
+    upz="1"
+    joint_limit="0.53">
     <origin xyz="0.0 0.0 0.0" rpy="0 0 0" />
     <axis xyz="0 1 0" />
@@ -130,5 +131,6 @@
     upx="0"
     upy="0"
-    upz="1">
+    upz="1"
+    joint_limit="0.53">
     <origin xyz="0.0 0.0 0.0" rpy="0 0 0" />
     <axis xyz="0 1 0" />
@@ -152,5 +154,6 @@
     upx="0"
     upy="0"
-    upz="1">
+    upz="1"
+    joint_limit="0.53">
     <origin xyz="0.0 0.0 0.0" rpy="0 0 0" />
     <axis xyz="0 1 0" />
@@ -167,5 +170,5 @@
     color="Blue"
     area="0.02"
-    control_joint_rad_to_cl="-4.0"
+    control_joint_rad_to_cl="-0.5"
     a0="0.0"
     cpx="-0.5"
@@ -174,5 +177,6 @@
     upx="0"
     upy="1"
-    upz="0">
+    upz="0"
+    joint_limit="0.53">
     <origin xyz="0.0 0.0 0.0" rpy="0 0 0" />
     <axis xyz="0 0 1" />
